Commit message: .

File: urdf/360_Camera_Model.urdf (robot description, URDF)
Before this commit: robot 360_Camera_Model, 5 links, 4 joints
Links:
- added link base_link, mass 0.19268; collision box size=0.1 0.1 0.1; visual box size=0.1 0.1 0.1
- link Rotator_1: mass 0.211155297251793 -> 0.211155
- link Rotator_2: mass 0.239977822875698 -> 0.239977
- link Rotator_3: mass 0.0829452509097665 -> 0.082945
Joints:
- removed joint Rotator_1_joint
- removed joint Rotator_2_joint
- removed joint Rotator_3_joint
- added joint Rotator_1_to_Fixed_base: type continuous, parent Fixed_base, child Rotator_1, origin xyz=0 0 0 rpy=0 0 0, axis 0 0 1, limit lower=0 upper=6.28319 effort=10 velocity=1
- added joint Rotator_2_to_Rotator_1: type revolute, parent Rotator_1, child Rotator_2, origin xyz=0.070003 0 -0.096227 rpy=0 0 0, axis 1 1 1, limit lower=0 upper=3.14159 effort=10 velocity=1
- added joint Rotator_3_to_Rotator_2: type revolute, parent Rotator_2, child Rotator_3, origin xyz=-0.07 0.040958 0 rpy=0 0 0, axis 1 1 1, limit lower=0 upper=1.5708 effort=1 velocity=1
- added joint fixed_base_to_base_link: type fixed, parent world, child Fixed_base, origin xyz=0 0 0 rpy=0 0 0
- joint base_to_world: child Fixed_base -> base_link
